Commit message: no commit

File: src/hector_quadrotor/hector_quadrotor_description/urdf/quadrotor.gazebo.xacro (robot description, xacro)
@@ -3,4 +3,3 @@
     <xacro:include filename="$(find hector_quadrotor_description)/urdf/quadrotor.urdf.xacro" />
     <xacro:include filename="$(find hector_quadrotor_gazebo)/urdf/quadrotor_plugins.gazebo.xacro" />
-    <!--<xacro:include filename="$(find hector_quadrotor_description)/urdf/quadrotor.gazebo.urdf.xacro" />-->
 </robot>

File: src/hector_quadrotor/hector_quadrotor_description/urdf/quadrotor_base.urdf.xacro (robot description, xacro)
@@ -5,4 +5,10 @@
   <!-- Main quadrotor link -->
   <xacro:macro name="quadrotor_base_macro">
+    <!--<link name="world"/>
+    <joint name="virtual_joint" type="floating">
+      <origin rpy="0 0 0" xyz="0 0 0"/>
+      <parent link="world"/>
+      <child link="base_link"/>
+    </joint>-->
     <link name="base_link">
       <inertial>

File: src/panda/panda_description/urdf/panda_arm.xacro (robot description, xacro)
@@ -16,5 +16,4 @@
       <parent link="world"/>
       <child link="${arm_id}_link0"/>
-      <!-- <origin xyz="0.0 0.0 0.0" rpy="0.0 0.0 0.0" /> -->
     </joint>
     <!-- Link 0 -->
